File: hardware/decoders/Atlas-N-1A-2-GP40-1/Atlas-N-1A-2-GP40-1.kicad_pcb (KiCad board)
At the start: 4 copper layers, 9 x 61.3 mm, 48 parts, among them J81 MCLR, J82 +5V, J83 GND, J84 PGD, J85 PGC, J86 RLP, J87 RLP, J88 RLP, J89 RLP, J90 RRP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

Commit message: Small corrections.
Parts:
- R55, R56, R59, R61, R62: value 390R -> 330R
- R57, R58: value 3K -> 3K3
