File: hardware/decoders/Atlas-N-1A-2-GP40-1/Atlas-N-1A-2-GP40-1.kicad_sch (KiCad schematic)
At the start: 48 parts, among them J81 MCLR, J82 +5V, J83 GND, J84 PGD, J85 PGC, J86 RLP, J87 RLP, J88 RLP, J89 RLP, J90 RRP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

Commit message: Small corrections.
Parts:
- C12, C13, C51, C52: Cost 0.01 -> 0.0697; MPN Generic -> GRM21BR61H106KE43L
- C21, C22: Cost 0.01 -> 0.0009; LCSC C49678 -> C1525; MPN Generic -> CL05B104KO5NNNC; Specification 0805 50V 100nF X7R 10% -> 402 16V 100nF X7R 10%
- D11, D12, D13, D14, D15, D21: Cost 0.01 -> 0.0119
- D61, D62: Cost 0.01 -> 0.0148
- J81, J82, J83, J84, J85, J86, J87, J88, J89, J90, J91, J92, J93, J94, J95: LCSC (none) -> DNP; MPN (none) -> DNP; Specification (none) -> 1.5mm x 3mm exposed pad.
- R21, R31, R32, R51, R52, R53, R54: LCSC C17414 -> C25744; MPN Generic -> 0402WGF1502TCE; Specification 0805 10K Ω 1% 1/8W -> 0402 15K Ω 1% 1/16W
- R55, R56, R59, R61, R62: value 390R -> 330R; LCSC C17655 -> C25104; MPN Generic -> 0402WGF3300TCE; Specification 0805 390 Ω 1% 1/8W -> 0403 330 Ω 1% 1/16W
- R57, R58: value 3K -> 3K3; LCSC C17661 -> C25890; MPN Generic -> 0402WGF3301TCE; Specification 0805 3K Ω 1% 1/8W -> 0402 3.3K Ω 1% 1/16W
- U21: value PIC18F06Q40-x/REB -> PIC18F16Q40-x/REB; LCSC (none) -> C3216898; MPN (none) -> PIC18F16Q40-I/REB
- U51: LCSC (none) -> C460274; MPN (none) -> ZXMHC6A07N8TC; Specification (none) -> SO-8 Full Bridge
